File: M.2-pcie-2x-adapter.kicad_pcb (KiCad board)
At the start: 4 copper layers, 100 x 95.5 mm, 32 parts, among them J1 Connector_PCIe_x4, U1 SY8204, U2 M.2-NGFF-Full

Commit message: Prepare for production
Parts:
- added H7: MountingHole, ToolingHole:ToolingHole_JLCSMT, F.Cu at (57.0, 10.3)
- added H8: MountingHole, ToolingHole:ToolingHole_JLCSMT, F.Cu at (152.9, 93.5)
Routing:
- net GND: vias 249 -> 248
- net (no net): vias 1 -> 0
Other:
- board text added: "JLCJLCJLCJLC"
